Commit message: Main

File: description/robot.urdf.xacro (robot description, xacro)
@@ -1,5 +1,4 @@
 <?xml version="1.0"?>
-<robot xmlns:xacro="http://www.ros.org/wiki/xacro"  name="B5_Rover">
-    <!-- Example link -->
-    <link name="base_link"></link>
+<robot xmlns:xacro="http://www.ros.org/wiki/xacro"  name="b5_rover">
+    <xacro:include filename="robot_core.xacro" />
 </robot>
